File: ledB/ledB.kicad_pcb (KiCad board)
At the start: 2 copper layers, 9 parts, among them U1 LMV321, Y1 Piezo Crystal

Commit message: rounded
Parts:
- removed D1: LED, LED_THT:LED_D3.0mm
- removed R1, R2, R3: 10M, Resistor_SMD:R_0805_2012Metric
- removed R4: 220, Resistor_SMD:R_0805_2012Metric
- added 10M: 10M, Resistor_THT:R_Axial_DIN0207_L6.3mm_D2.5mm_P10.16mm_Horizontal, F.Cu at (122.6, 140.0)
- added 10k: 10K, Resistor_THT:R_Axial_DIN0207_L6.3mm_D2.5mm_P10.16mm_Horizontal, F.Cu at (134.6, 135.1)
- added Diode: 1N4001, Diode_THT:D_DO-41_SOD81_P10.16mm_Horizontal, F.Cu at (120.0, 125.1)
- added G***: LOGO, logo:TAMI_logo, F.Cu at (127.5, 114.3)
- BT1: value Battery Cell -> Battery_Cell; footprint Connector_Wire:SolderWire-2.5sqmm_1x02_P7.2mm_D2.4mm_OD3.6mm -> 1_my_custom_lib:BAT_BH800S; moved to B.Cu
- U1: value LMV321 -> LM741C; footprint Package_TO_SOT_SMD:SOT-23-5_HandSoldering -> Package_DIP:DIP-8_W7.62mm
- Y1: value Piezo Crystal -> Crystal; moved to B.Cu
- moved D2 175.5 mm to (128.9, 122.6), turned to 180 degrees
- moved BT1 46.6 mm to (127.6, 131.5), turned to 0 degrees
- moved U1 41.1 mm to (131.4, 135.3), turned to 180 degrees
- moved Y1 11.8 mm to (126.4, 111.8), turned to -90 degrees
Connections:
- D2 pad 1: unconnected-(D2-K-Pad1) -> GND
- D2 pad 2: unconnected-(D2-A-Pad2) -> Net-(D1-K)
- U1 pad 1: Net-(U1-+) -> unconnected-(U1-NULL-Pad1)
- U1 pad 2: GND -> PIEZO+
- U1 pad 3: Net-(U1--) -> Net-(U1-+)
- U1 pad 4: Net-(R2-Pad1) -> GND
- U1 pad 5: VCC -> unconnected-(U1-NULL-Pad5)
- Y1 pad 2: Net-(U1--) -> PIEZO+
Routing:
- net GND: track 45.2 -> 0.00 mm
- net PIEZO+: track 0.00 -> 29.9 mm
- net Net-(R2-Pad1): track 18.4 -> 0.00 mm
- net Net-(U1--): track 16.5 -> 0.00 mm
- net Net-(U1-+): track 17.5 -> 6.02 mm
- net Net-(D1-K): track 0.00 -> 6.99 mm
- net VCC: track 22.4 -> 16.2 mm
- net Net-(D1-A): track 14.8 -> 12.0 mm
- added copper zone on F.Cu, net GND
Other:
- board outline added: 24.1 x 34.9 mm
- board text added: "Genuine TI LM741C only"
- board text added: "LED"
- board text added: "LED-B"
