File: ledB/ledB.kicad_pcb (KiCad board)
At the start: 2 copper layers, 9 parts, among them U1 LMV321, Y1 Piezo Crystal

Commit message: sent to fab
Parts:
- removed BT1: Battery Cell, Connector_Wire:SolderWire-2.5sqmm_1x02_P7.2mm_D2.4mm_OD3.6mm
- removed D2: LED, LED_THT:LED_D3.0mm
- added ?: , , F.Cu at (110.5, 137.0)
- added ?: , , F.Cu at (110.5, 116.5)
- added H1: MountingHole, MountingHole:MountingHole_3.5mm, F.Cu at (110.5, 108.0)
- added TP2: TestPoint, TestPoint:TestPoint_Pad_2.0x2.0mm, F.Cu at (112.0, 124.0)
- moved R3 38.4 mm to (115.0, 129.4), turned to 90 degrees
- moved R4 35.6 mm to (106.0, 124.5), turned to 0 degrees
- moved U1 34.6 mm to (110.0, 128.5), turned to -90 degrees
- moved R2 30.6 mm to (104.5, 129.1), turned to 90 degrees
- moved R1 25.3 mm to (115.0, 123.6), turned to 90 degrees
- moved D1 24.0 mm to (111.3, 120.0), turned to 180 degrees
- moved Y1 19.1 mm to (112.0, 113.0), turned to -90 degrees
Connections:
- net Net-(U1--) renamed /piezo+
Routing:
- net GND: track 45.2 -> 10.1 mm
- net Net-(D1-A): track 14.8 -> 5.25 mm
- net Net-(U1-+): track 17.5 -> 11.5 mm
- net /piezo+: track 16.5 -> 22.3 mm, vias 0 -> 1
- net Net-(R2-Pad1): track 18.4 -> 12.5 mm
- net VCC: track 22.4 -> 23.4 mm
- added copper zone on F.Cu, net GND
Other:
- board outline added: 24.1 x 34.9 mm
- board text added: "Was würde Uwe tun ?"
- board text added: "piezo"

Commit message: v2 based on ledman
Parts:
- removed TP2: TestPoint, TestPoint:TestPoint_Pad_2.0x2.0mm
- added 47n: 47n, Capacitor_SMD:C_0805_2012Metric, F.Cu at (112.0, 124.0)
- 2M2: renamed from R1; value 10M -> 2M2
- 3M3: renamed from R2; value 10M -> 3M3
- 3M3: renamed from R3; value 10M -> 3M3
- moved D1 14.0 mm to (111.3, 134.0)
- moved 220 9.05 mm to (105.1, 133.5)
- moved H1 0.50 mm to (110.5, 107.5)
- renumbered R4 to 220, U1 to LMV321
Routing:
- net GND: track 10.1 -> 0.71 mm
- net Net-(R2-Pad1): track 12.5 -> 7.75 mm
- net Net-(D1-A): track 5.25 -> 2.94 mm
- net /piezo+: track 22.3 -> 20.7 mm, vias 1 -> 0

Commit message: diy ledman
Parts:
- removed ? (x2): , 
- removed D1: LED, LED_THT:LED_D3.0mm
- removed H1: MountingHole, MountingHole:MountingHole_3.5mm
- removed Y1: Piezo Crystal, Connector_PinHeader_2.54mm:PinHeader_1x02_P2.54mm_Vertical
Routing:
- net GND: track 0.71 -> 10.3 mm
- net VCC: track 23.4 -> 27.9 mm
- net /piezo+: track 20.7 -> 16.3 mm
- removed copper zone on F.Cu, net GND
Other:
- board size 24.1 x 34.9 mm -> 26 x 34 mm
- board text added: "LED+"
- board text added: "PIEZO +"
- board text removed: "Was würde Uwe tun ?"

Commit message: etch
Routing:
- net GND: track 10.3 -> 18.4 mm
